File: My Projects.kicad_sch (KiCad schematic)
At the start: 4 parts, among them IC1 7483, IC2 7483, IC3 7486, IC4 7486

Commit message: ..
Parts:
- added SW1, SW2, SW3, SW4, SW5, SW6, SW7, SW8: SW_SPST, symbol Switch:SW_SPST
Connections:
- net B7: now reaches IC3.1
- net B4: now reaches IC3.12
- net B6: now reaches IC3.4
- net B5: now reaches IC3.9
- net B3: now reaches IC4.1
- net B0: now reaches IC4.12
- net B2: now reaches IC4.4
- net B1: now reaches IC4.9
