File: My Projects.kicad_sch (KiCad schematic)
At the start: 68 parts, among them IC1 7483, IC2 7483, IC3 7486, IC4 7486, SW1 SW_SPST, SW10 SW_SPST, SW11 SW_SPST, SW12 SW_SPST, SW13 SW_SPST, SW14 SW_SPST, SW15 SW_SPST, SW16 SW_SPST, SW2 SW_SPST, SW3 SW_SPST, SW4 SW_SPST, SW5 SW_SPST, SW6 SW_SPST, SW7 SW_SPST, SW8 SW_SPST, SW9 SW_SPST

Commit message: COMMIT
Parts:
- IC1: footprint (none) -> Package_DIP:DIP-16_W10.16mm
- IC4: footprint (none) -> Package_DIP:DIP-14_W10.16mm
Changed lines of the file:
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@@
 			)
 		)
-		(property "Footprint" ""
+		(property "Footprint" "Package_DIP:DIP-14_W10.16mm"
 			(at 199.39 72.39 0)
 			(effects
@@
 			)
 		)
-		(property "Footprint" ""
+		(property "Footprint" "Package_DIP:DIP-16_W10.16mm"
 			(at 102.87 120.65 0)
 			(effects
